Commit message: better driving performance

File: simulation/assets/robots/house_bot/robot.urdf (robot description, URDF)
Before this commit: robot house_bot, 5 links, 4 joints
Links:
- link base_link: geometry visual mesh filename=meshes/chassis.obj

File: simulation/assets/robots/mr_stabs_mk2/robot.urdf (robot description, URDF)
Before this commit: robot mr_stabs_mk2, 3 links, 2 joints
Links:
- added link caster_front, mass 0.001; collision sphere radius=0.005
- added link caster_rear, mass 0.001; collision sphere radius=0.005
- link base_link: geometry visual mesh filename=meshes/chassis.obj
Joints:
- added joint caster_front_joint: type fixed, parent base_link, child caster_front, origin xyz=0.08 0.0 -0.020 rpy=0 0 0
- added joint caster_rear_joint: type fixed, parent base_link, child caster_rear, origin xyz=-0.015 0.0 -0.020 rpy=0 0 0

Commit message: good physics and frame rate performance

File: simulation/assets/robots/house_bot/robot.urdf (robot description, URDF)
Before this commit: robot house_bot, 5 links, 4 joints
Joints:
- joint front_left_wheel_joint: origin xyz=1.0000000000e-01 1.0000000000e-01 0.0000000000e+00 rpy=0 0 0 -> xyz=1.0000000000e-01 1.0000000000e-01 -8.3000000000e-02 rpy=0 0 0
- joint front_right_wheel_joint: origin xyz=1.0000000000e-01 -1.0000000000e-01 0.0000000000e+00 rpy=0 0 0 -> xyz=1.0000000000e-01 -1.0000000000e-01 -8.3000000000e-02 rpy=0 0 0
- joint rear_left_wheel_joint: origin xyz=-1.0000000000e-01 1.0000000000e-01 0.0000000000e+00 rpy=0 0 0 -> xyz=-1.0000000000e-01 1.0000000000e-01 -8.3000000000e-02 rpy=0 0 0
- joint rear_right_wheel_joint: origin xyz=-1.0000000000e-01 -1.0000000000e-01 0.0000000000e+00 rpy=0 0 0 -> xyz=-1.0000000000e-01 -1.0000000000e-01 -8.3000000000e-02 rpy=0 0 0
