Commit message: add experiment files. fix quaternion conversion issue

File: simulation/assets/robots/mr_stabs_mk2/robot.urdf (robot description, URDF)
Before this commit: robot mr_stabs_mk2, 5 links, 4 joints
Joints:
- joint caster_rear_joint: origin xyz=-0.015 0.0 -0.020 rpy=0 0 0 -> xyz=-0.08 0.0 -0.020 rpy=0 0 0

Commit message: fix simulation dynamics

File: simulation/assets/robots/mr_stabs_mk2/robot.urdf (robot description, URDF)
Before this commit: robot mr_stabs_mk2, 5 links, 4 joints
Links:
- link caster_front: geometry collision sphere radius=0.001
- link caster_rear: geometry collision sphere radius=0.001
