File: hardware/mr_stabs_mk2_pcb/pcba/mk2_sch_imu_and_radio.kicad_sch (KiCad schematic)
At the start: 11 parts, among them U4 BNO055, Y1 32.768kHz

Commit message: Re-route the Mk2 board at JLCPCB's 2 oz rules and fit the CPL rotations
The board orders with 2 oz outer copper, but it was routed at 0.15 mm clearance, a 1 oz
number. Against JLCPCB's 2 oz minimums (0.16 mm track, 0.20 mm space) it had 292 violations
behind a clean DRC. Re-routed at 0.20 mm: 0 errors, 0 unconnected, with mk2_routed.kicad_dru
holding the 2 oz rules so the KiCad GUI checks the same thing.

Getting the stem to route at 0.20 mm took these changes:
- Signal vias 0.5 / 0.25 mm; GND, battery and 5 V vias stay 0.6 / 0.3. Min hole 0.25 mm.
- C3 (100 uF bulk) back on the right ear beside the shunt. Its feed across the stem never
  routed at 2 oz spacing, and a prewired track there walled off the signals. It gives up the
  stem's protection from a dislodged motor.
- INA238 VBUS on BAT_IN, the F pour under the pin. Reads the shunt drop high, at most 35 mV at
  a 70 A stall; current sensing is unchanged.
- B keepouts hold the VBATT pour's neck (shunt to ESC_L+) and R3's Kelvin tap open: signal
  tracks had split the pour and left the ESC current on a track.
- F VBATT patch over the buck input, with the B VBATT pour extended under it so every piece
  stitches down. C6 turned to face it; INA238 moved 0.3 mm off the rear edge.

The copper IR solve now gives a 23.8 mV VBATT drop at 70 A, down from 42.4 mV.

cpl.csv angles and centres are fitted to JLCPCB's own footprint for each LCSC number
(cpl_check.csv). KiCad's angles would have placed C3 reversed and five ICs 90 degrees out.
R5 and U5 no longer have vias in their pads; C14 and C10 still do (open question 8).

Co-Authored-By: Claude Opus 5.5 <noreply@anthropic.com>
Parts:
- removed C20: 100nF, symbol Device:C
- added H2: NANO_RX, symbol mk2:HXPZ2.54-1X4PWT
- C21: renamed from H2; value NANO_RX -> 100nF; symbol mk2:HXPZ2.54-1X4PWT -> Device:C
- renumbered C21 to C20
Connections:
- net +3V3: now also C21.1
- net +5V: now also H2.2; no longer C21.2
- net CRSF_RX_RX: now also H2.4; no longer C21.4
- net CRSF_RX_TX: now also H2.3; no longer C21.3
- net GND: now also C21.2, H2.1; no longer C21.1
Other:
- moved on the sheet: C20
