File: hardware/mr_stabs_mk2_pcb/pcba/mk2_sch_mcu_and_usb.kicad_sch (KiCad schematic)
At the start: 21 parts, among them U5 USBLC6-2SC6

Commit message: Re-route the Mk2 board at JLCPCB's 2 oz rules and fit the CPL rotations
The board orders with 2 oz outer copper, but it was routed at 0.15 mm clearance, a 1 oz
number. Against JLCPCB's 2 oz minimums (0.16 mm track, 0.20 mm space) it had 292 violations
behind a clean DRC. Re-routed at 0.20 mm: 0 errors, 0 unconnected, with mk2_routed.kicad_dru
holding the 2 oz rules so the KiCad GUI checks the same thing.

Getting the stem to route at 0.20 mm took these changes:
- Signal vias 0.5 / 0.25 mm; GND, battery and 5 V vias stay 0.6 / 0.3. Min hole 0.25 mm.
- C3 (100 uF bulk) back on the right ear beside the shunt. Its feed across the stem never
  routed at 2 oz spacing, and a prewired track there walled off the signals. It gives up the
  stem's protection from a dislodged motor.
- INA238 VBUS on BAT_IN, the F pour under the pin. Reads the shunt drop high, at most 35 mV at
  a 70 A stall; current sensing is unchanged.
- B keepouts hold the VBATT pour's neck (shunt to ESC_L+) and R3's Kelvin tap open: signal
  tracks had split the pour and left the ESC current on a track.
- F VBATT patch over the buck input, with the B VBATT pour extended under it so every piece
  stitches down. C6 turned to face it; INA238 moved 0.3 mm off the rear edge.

The copper IR solve now gives a 23.8 mV VBATT drop at 70 A, down from 42.4 mV.

cpl.csv angles and centres are fitted to JLCPCB's own footprint for each LCSC number
(cpl_check.csv). KiCad's angles would have placed C3 reversed and five ICs 90 degrees out.
R5 and U5 no longer have vias in their pads; C14 and C10 still do (open question 8).

Co-Authored-By: Claude Opus 5.5 <noreply@anthropic.com>
Parts:
- removed C2: 100nF, symbol Device:C
- added USB1: TYPE-C-31-D-06, symbol mk2:TYPE-C-31-D-06
- C15: renamed from USB1; value TYPE-C-31-D-06 -> 10uF; symbol mk2:TYPE-C-31-D-06 -> Device:C
- C2: renamed from C15; value 10uF -> 100nF
Connections:
- net +3V3: now also C15.1
- net GND: now also C15.2, USB1.A1 (GND), USB1.A12 (GND), USB1.B1 (GND), USB1.B12 (GND), USB1.EP; no longer C15.A1 (GND), C15.A12 (GND), C15.B1 (GND), C15.B12 (GND), C15.EP
- net at ESP1.24 (IO20), U5.1 (I/O1), U5.6 (I/O1): now also USB1.A6 (DP1), USB1.B6 (DP2); no longer C15.A6 (DP1), C15.B6 (DP2)
- net at ESP1.23 (IO19), U5.3 (I/O2), U5.4 (I/O2): now also USB1.A7 (DN1), USB1.B7 (DN2); no longer C15.A7 (DN1), C15.B7 (DN2)
- net at R15.1: now also USB1.A5 (CC1); no longer C15.A5 (CC1)
- net at R16.1: now also USB1.B5 (CC2); no longer C15.B5 (CC2)
- new net: D2.2 (A), U5.5 (VBUS), USB1.A4 (VBUS), USB1.A9 (VBUS), USB1.B4 (VBUS), USB1.B9 (VBUS)
Other:
- moved on the sheet: C2
